Commit message: Add RGBD camera

File: src/my_robot/urdf/my_robot.xacro (robot description, xacro)
@@ -126,5 +126,5 @@
         <dynamics damping="1.0" friction="1.0" />
     </joint>
-    <!-- Camera -->
+    <!-- RGBD Camera -->
     <link name="camera">
         <xacro:cube_inertial mass="${camera_mass}" edge_length="${camera_edge_length}" />
@@ -148,4 +148,11 @@
         <axis xyz="0 1 0" rpy="0 0 0" />
     </joint>
+    <joint name="camera_optical_joint" type="fixed">
+        <origin xyz="0 0 0" rpy="${-pi/2} 0 ${-pi/2}"/>
+        <parent link="camera"/>
+        <child link="camera_link_optical"/>
+    </joint>
+    <link name="camera_link_optical">
+    </link>
     <!-- Lidar -->
     <link name="hokuyo">

Commit message: Correct topics and robot_footprint
Now building should be changed by something smaller/with
more obstacles and then map generated by running our robot
around

File: src/my_robot/urdf/my_robot.xacro (robot description, xacro)
@@ -148,4 +148,5 @@
         <axis xyz="0 1 0" rpy="0 0 0" />
     </joint>
+    <link name="camera_link_optical"></link>
     <joint name="camera_optical_joint" type="fixed">
         <origin xyz="0 0 0" rpy="${-pi/2} 0 ${-pi/2}"/>
@@ -153,6 +154,4 @@
         <child link="camera_link_optical"/>
     </joint>
-    <link name="camera_link_optical">
-    </link>
     <!-- Lidar -->
     <link name="hokuyo">
