Commit message: Rename package and correct teleop launch file
Most likely teleop launch file's location will be changed
to be inside teleop package itself

File: src/slamming_robot/urdf/slamming_robot.xacro (robot description, xacro)
@@ -1,4 +1,4 @@
 <?xml version="1.0"?>
-<robot name="my_robot" xmlns:xacro="http://www.ros.org/wiki/xacro">
+<robot name="slamming_robot" xmlns:xacro="http://www.ros.org/wiki/xacro">
     <!-- CONSTANTS -->
     <xacro:property name="pi" value="3.1415926535897931" />
@@ -30,7 +30,7 @@
     <xacro:property name="sensors_base_offset_z" value="${base_height/2 + sensors_base_heigth/2}" />
     <!-- INCLUDES -->
-    <xacro:include filename="$(find my_robot)/urdf/materials.xacro" />
-    <xacro:include filename="$(find my_robot)/urdf/macros.xacro" />
-    <xacro:include filename="$(find my_robot)/urdf/my_robot.gazebo" />
+    <xacro:include filename="$(find slamming_robot)/urdf/materials.xacro" />
+    <xacro:include filename="$(find slamming_robot)/urdf/macros.xacro" />
+    <xacro:include filename="$(find slamming_robot)/urdf/slamming_robot.gazebo" />
     <!-- ROBOT DESCRIPTION-->
     <link name="robot_footprint"></link>
@@ -166,5 +166,5 @@
             <origin xyz="0 0 0" rpy="0 0 0" />
             <geometry>
-                <mesh filename="package://my_robot/meshes/hokuyo.dae" />
+                <mesh filename="package://slamming_robot/meshes/hokuyo.dae" />
             </geometry>
         </visual>

Commit message: Make joint between basis and sensor basis fixed
Sensor basis is rotating with sudden changes of direction
and that's affecting the mapping process, because the sensors
stop being aligned with the wheels

File: src/slamming_robot/urdf/slamming_robot.xacro (robot description, xacro)
@@ -118,5 +118,5 @@
         </visual>
     </link>
-    <joint name="sensors_base_hinge" type="continuous">
+    <joint name="sensors_base_suture" type="fixed">
         <origin xyz="0 0 ${sensors_base_offset_z}" rpy="0 0 0" />
         <child link="sensors_base" />
